Commit message: new name for the node robot state publisher in the launch display

File: cc8_description/urdf/cc8.xacro (robot description, xacro)
@@ -187,6 +187,6 @@
       </geometry>
       <material name="silver"/>
-    <!--</visual>
-    <collision>
+    </visual>
+    <!--<collision>
       <origin xyz="0.503097 -0.414731 -0.025175" rpy="0 0 0"/>
       <geometry>
@@ -367,4 +367,5 @@
     </collision>
   </link>
+<!--ZED 2i Joint-->
   <joint name="zed2_camera_center_joint" type="fixed">
     <parent link="base_link"/>
@@ -372,11 +373,9 @@
     <origin xyz="0.39 0 0.09" rpy="0 0 0"/>
   </joint>
-  <!--<xacro:if value="${footprint_link}">-->
-    <joint name="base_joint" type="fixed">
-      <origin xyz="0 0 0.25" rpy="0 0 0"/>
-      <parent link="base_footprint"/>
-      <child link="base_link"/>
-    </joint>
-  <!--</xacro:if>-->
+  <joint name="base_joint" type="fixed">
+    <origin xyz="0 0 0.25" rpy="0 0 0"/>
+    <parent link="base_footprint"/>
+    <child link="base_link"/>
+  </joint>
   <joint name="fixed_joint_L" type="fixed">
     <origin xyz="0.0 0.275 0.15" rpy="0 0 0"/>
